File: schematic/1_bit_adder.kicad_sch (KiCad schematic)
At the start: 39 parts, among them Q1 2N7000, Q10 2N7000, Q11 2N7000, Q12 2N7000, Q13 2N7000, Q14 2N7000, Q15 2N7000, Q16 2N7000, Q17 2N7000, Q18 2N7000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

Commit message: minor
Parts:
- R1, R10, R11, R12, R2, R3, R4, R5, R6, R7, R8, R9: value R -> 1k
Changed lines of the file:
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@@
 			)
 		)
-		(property "Value" "R"
+		(property "Value" "1k"
 			(at 125.73 113.0299 0)
 			(effects
@@
 			)
 		)
-		(property "Value" "R"
+		(property "Value" "1k"
 			(at 227.33 113.0299 0)
 			(effects
@@
 	)
 	(symbol
+		(lib_name "74HC00_1")
 		(lib_id "74xx:74HC00")
 		(at 99.06 60.96 0)
@@
 			)
 		)
-		(property "Value" "R"
+		(property "Value" "1k"
 			(at 30.48 149.86 90)
 			(effects
@@
 			)
 		)
-		(property "Value" "R"
+		(property "Value" "1k"
 			(at 201.93 113.0299 0)
 			(effects
@@
 			)
 		)
-		(property "Value" "R"
+		(property "Value" "1k"
 			(at 252.73 113.0299 0)
 			(effects
@@
 			)
 		)
-		(property "Value" "R"
+		(property "Value" "1k"
 			(at 74.93 113.0299 0)
 			(effects
@@
 			)
 		)
-		(property "Value" "R"
+		(property "Value" "1k"
 			(at 176.53 113.0299 0)
 			(effects
@@
 			)
 		)
-		(property "Value" "R"
+		(property "Value" "1k"
 			(at 49.53 113.0299 0)
 			(effects
@@
 			)
 		)
-		(property "Value" "R"
+		(property "Value" "1k"
 			(at 30.48 137.16 90)
 			(effects
@@
 			)
 		)
-		(property "Value" "R"
+		(property "Value" "1k"
 			(at 100.33 113.0299 0)
 			(effects
@@
 			)
 		)
-		(property "Value" "R"
+		(property "Value" "1k"
 			(at 151.13 113.0299 0)
 			(effects
@@
 			)
 		)
-		(property "Value" "R"
+		(property "Value" "1k"
 			(at 30.48 124.46 90)
 			(effects
