File: schematic/1_bit_register.kicad_sch (KiCad schematic)
At the start: 57 parts, among them Q1 BS250, Q10 2N7000, Q11 2N7000, Q12 2N7000, Q13 2N7000, Q14 2N7000, Q15 2N7000, Q16 2N7000, Q17 2N7000, Q18 2N7000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

Commit message: sim circuit for register
Connections:
- net at Q23.3 (S), Q24.3 (D), Q5.2 (G)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: no longer Q10.3 (D), Q13.2 (G), Q14.2 (G), Q17.2 (G), R10.2
- net at U0.3, U1.1: now also U10.2, U9.1; no longer U8.1, U9.2
- net at U5.3, U6.1: now also U8.1, U9.2; no longer U10.2, U9.1
- new net: Q10.3 (D), Q13.2 (G), Q14.2 (G), Q17.2 (G), R10.2
