File: schematic/clock.kicad_sch (KiCad schematic)
At the start: 26 parts, among them Q1 2N7000

Commit message: clock component schematic
Parts:
- added C2, C4: 0.1mF, symbol Device:C
- added C3: 1mF, symbol Device:C
- added D2: ~, symbol Device:LED
- added Q12, Q14, Q15, Q16, Q17, Q18, Q19, Q2, Q28, Q29, Q3, Q30, Q32, Q33, Q34, Q35, Q36, Q37, Q38, Q39, Q40, Q41, Q43, Q9: 2N7000, Package_TO_SOT_THT:TO-92_Inline, symbol Transistor_FET:2N7000
- added Q20, Q21, Q22, Q23, Q24, Q25, Q26, Q27, Q31, Q42: BS250, Package_TO_SOT_THT:TO-92_Inline, symbol Transistor_FET:BS250
- added R16, R20, R23, R26, R31, R32, R33: 4.7k, symbol Device:R
- added R21, R24, R27, R28, R29, R30, R37, R38, R39, R40, R41, R42, R43, R44, R45, R46, R47, R48, R51, R52: 1k, symbol Device:R
- added R22, R25, R36, R50: 10k, symbol Device:R
- added R34: 150, symbol Device:R
- added R35: 3M, symbol Device:R
- added R49: 2.2k, symbol Device:R
- added R53, R54: 100k, symbol Device:R
- added SW3: ~, symbol Switch:SW_SP3T
- added SW4: SW_MEC_5E, symbol Switch:SW_MEC_5E
Connections:
- net +5V: now also R16.1, R20.1, R21.1, R23.1, R24.1, R26.1, R27.1, R28.1, R29.1, R30.1, R31.1, R34.1, R37.1, R38.1, R40.1, R41.1, R42.1, R43.1, R44.1, R45.1, R46.1, R47.1, R51.1
- net GND: now also C2.2, C3.2, C4.2, D2.1 (K), Q14.1 (S), Q16.1 (S), Q18.1 (S), Q19.1 (S), Q22.1 (D), Q26.1 (D), Q28.1 (S), Q29.1 (S), Q33.1 (S), Q34.1 (S), Q35.1 (S), Q37.1 (S), Q38.1 (S), Q39.1 (S), Q40.1 (S), Q41.1 (S), R22.2, R25.2, R33.2, R39.2, R48.2, R50.1, R53.2, R54.2
- net clock_out: now also Q42.1 (D), Q43.3 (D)
- net at SW1.1: now also U10.2, U8.1; no longer R18.1
- net at SW1.2: now also R18.1; no longer R19.1
- removed net auto_timer_en: SW1.4, U10.2, U8.1
- new net: C3.1, Q28.3 (D), Q3.2 (G), Q9.2 (G), R35.2, R36.2
- new net: Q12.3 (D), Q26.2 (G), Q27.1 (D), Q27.2 (G)
- new net: Q25.3 (S), Q26.3 (S), R24.2
- new net: Q41.3 (D), Q42.2 (G), Q43.2 (G), R46.2, R49.1
- new net: C4.1, Q36.2 (G), R52.2
- new net: C2.1, Q12.2 (G), R32.2, R33.1
- new net: Q16.2 (G), Q17.3 (D), Q28.2 (G), R29.2
- new net: Q15.1 (S), Q16.3 (D)
- new net: R34.2, SW3.3
- new net: Q32.1 (S), Q33.3 (D)
- new net: Q32.2 (G), Q35.3 (D), R42.2
- new net: Q32.3 (D), Q34.2 (G), R40.2
- new net: Q42.3 (S), R47.2
- new net: Q14.2 (G), Q21.1 (D), R53.1
- new net: Q14.3 (D), Q15.2 (G), R27.2
- new net: Q36.3 (D), Q38.2 (G), R43.2
- new net: Q38.3 (D), Q39.2 (G), R44.2
- new net: Q19.2 (G), Q25.1 (D)
- new net: Q24.1 (D), Q24.2 (G), Q25.2 (G), Q9.3 (D)
- new net: Q35.2 (G), Q37.2 (G), R54.1, SW3.4
- new net: D2.2 (A), R49.2
- new net: Q2.3 (D), Q20.1 (D), Q20.2 (G), Q21.2 (G)
- new net: Q20.3 (S), R16.2
- new net: R19.1, SW1.4
- new net: Q31.3 (S), R38.2
- new net: Q34.3 (D), Q40.2 (G), R41.2
- new net: Q18.2 (G), Q19.3 (D), R30.2
- new net: Q17.1 (S), Q18.3 (D)
- new net: Q24.3 (S), R23.2
- new net: R36.1, SW3.1
- new net: Q30.3 (D), Q31.1 (D), Q33.2 (G)
- new net: Q29.3 (D), Q30.2 (G), Q31.2 (G), R37.2
- new net: Q23.3 (S), R20.2
- new net: Q21.3 (S), Q22.3 (S), R21.2
- new net: Q15.3 (D), Q17.2 (G), Q29.2 (G), R28.2
- new net: R51.2, SW4.4 (A)
- new net: R52.1, SW4.1
- new net: Q39.3 (D), Q40.3 (D), Q41.2 (G), R45.2
- new net: Q2.1 (S), Q3.1 (S), R22.1
- new net: Q2.2 (G), R31.2, R32.1
- new net: R50.2, SW4.2
- new net: Q22.2 (G), Q23.1 (D), Q23.2 (G), Q3.3 (D)
- new net: Q36.1 (S), Q37.3 (D)
- new net: Q12.1 (S), Q9.1 (S), R25.1
- new net: Q43.1 (S), R48.1
- new net: Q27.3 (S), R26.2
- new net: Q30.1 (S), R39.1
- new net: R35.1, SW3.2
Other:
- moved on the sheet: C1, D1, Q1, R13, R14, R15, R17, R18, R19, SW1, SW2, U10A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

Commit message: clock v2 schematic
Parts:
- removed D1, D2: ~, symbol Device:LED
- removed Q1, Q12, Q14, Q15, Q16, Q17, Q18, Q19, Q2, Q3, Q35, Q36, Q37, Q38, Q39, Q40, Q41, Q43, Q9: 2N7000, Package_TO_SOT_THT:TO-92_Inline, symbol Transistor_FET:2N7000
- removed Q20, Q21, Q22, Q23, Q24, Q25, Q26, Q27, Q31: BS250, Package_TO_SOT_THT:TO-92_Inline, symbol Transistor_FET:BS250
- removed R13, R14, R15, R17, R18, R19: ~, symbol Device:R
- removed R16, R20, R23, R26: 4.7k, symbol Device:R
- removed R21, R24, R27, R28, R29, R30: 1k, symbol Device:R
- removed R22, R25: 10k, symbol Device:R
- removed R34: 150, symbol Device:R
- removed R54: 100k, symbol Device:R
- removed SW1, SW3: ~, symbol Switch:SW_SP3T
- removed SW2: ~, symbol Switch:SW_DIP_x01
- removed SW4: SW_MEC_5E, symbol Switch:SW_MEC_5E
- removed U1, U10, U4, U9: ~, symbol 74xx:74HC00
- removed U11, U13, U15, U2, U5, U8: ~, symbol 74xx:74HC04
- removed U12: ~, symbol 74xx:7402
- removed U14, U3: ~, symbol 74xx:74LCX07
- removed U6, U7: ~, Package_BGA:Texas_DSBGA-8_1.5195x1.5195mm_Layout3x3_P0.5mm, symbol Comparator:LMV7272
- added C5: 100nF, symbol Device:C
- added D1, D2, D3, D4, D5, D6, D7: ~, Diode_THT:D_DO-41_SOD81_P10.16mm_Horizontal, symbol Diode:1N4001
- added D8: ~, symbol Device:LED
- added Q20, Q21, Q22, Q23, Q24, Q25, Q26, Q27, Q31: 2N7000, Package_TO_SOT_THT:TO-92_Inline, symbol Transistor_FET:2N7000
- added SW4: ~, symbol Switch:SW_SP3T
- added SW5: ~, symbol Switch:SW_MEC_5E
- C1: value C -> 68pF
- C2: value 0.1mF -> 68pF
- C3: value 1mF -> 10mF
- C4: value 0.1mF -> 10mF
- R31, R32: value 4.7k -> 1k
- R33: value 4.7k -> 100k
- R35: value 3M -> 100k
- R36: value 10k -> 1k
- R37, R38, R43, R44, R47: value 1k -> 100k
- R42: value 1k -> 2.2k
- R50: value 10k -> 2.2k
- R53: value 100k -> 1k
Connections:
- net +5V: now also Q42.3 (S), R32.1, R36.1, R39.1, R42.2, R45.2, R46.2, R48.2, R50.2, R51.2, R52.2, R53.2, SW4.3; no longer R37.1, R38.1, R40.1, R41.1, R42.1, R43.1, R44.1, R45.1, R46.1, R47.1, R51.1
- net GND: now also Q30.1 (S), Q32.1 (S), R41.1, R43.2, R44.2, R49.1, C5.1, D8.1 (K), Q20.1 (S), Q21.1 (S), Q22.1 (S), Q23.1 (S), Q25.1 (S), Q27.1 (S), Q31.1 (S); no longer C1.2, C2.2, C3.2, C4.2, Q28.1 (S), R33.2, R39.2, R48.2, R50.1, R53.2
- net clock_out: now also Q31.3 (D)
- net at C4.1: now also R37.1, D2.1 (K), Q22.3 (D); no longer R52.2
- net at C2.1, R33.1: now also D1.1 (K), Q20.3 (D); no longer R32.2
- net at Q28.2 (G): now also R32.2, D3.2 (A)
- net at Q33.3 (D): now also R52.1, D6.2 (A); no longer Q32.1 (S)
- net at Q32.2 (G): now also Q28.3 (D), R48.1; no longer R42.2
- net at R47.2: no longer Q42.3 (S)
- net at R53.1: now also Q34.3 (D), D7.2 (A)
- net at R49.2: now also Q30.2 (G), Q42.2 (G), D5.1 (K), D6.1 (K), D7.1 (K), Q31.2 (G)
- net at R38.2: now also C4.2, Q23.2 (G)
- net at R41.2: now also SW5.3 (K); no longer Q34.3 (D)
- net at C1.1: now also R33.2, Q20.2 (G)
- net at Q33.2 (G): now also R46.1, Q26.3 (D); no longer Q30.3 (D)
- net at Q29.2 (G): now also R47.1, SW4.1
- net at R31.2: now also D1.2 (A); no longer R32.1
- net at R35.1: now also C1.2, D3.1 (K), Q21.3 (D)
- new net: R42.1, SW5.1
- new net: R40.1, SW5.2
- new net: Q28.1 (S), Q29.3 (D)
- new net: C3.1, Q22.2 (G), R37.2
- new net: C2.2, Q21.2 (G), R35.2
- new net: Q27.2 (G), R44.1, SW4.2
- new net: Q26.1 (S), Q27.3 (D)
- new net: Q25.2 (G), R43.1, SW4.4
- new net: D4.2 (A), Q26.2 (G), R39.2
- new net: Q24.3 (D), Q34.2 (G), R45.1
- new net: C3.2, D4.1 (K), Q23.3 (D), R38.1
- new net: D2.2 (A), R36.2
- new net: D5.2 (A), Q32.3 (D), R51.1
- new net: C5.2, Q24.2 (G), R40.2
- new net: D8.2 (A), Q30.3 (D), R50.1
- new net: Q24.1 (S), Q25.3 (D)
Other:
- note added: "Fast clock (~100kHz)"
- note added: "Manual clock"
- note added: "Slow clock (~1Hz)"
- note removed: "automatic clock (like astable 555 timer)"
- note removed: "manual input"
- note removed: "output"
- note removed: "timing mode signal select"
- note removed: "timing select (fast, slow, manual)"
